File: hw/rj45/panel/rj45_panel.kicad_pcb (KiCad board)
At the start: 6 copper layers, 71.4 x 107 mm, 471 parts, among them J1 SFP edge (INF-8074i), J2 KH-RJ45-58-8P8C, T1 LP72450ANL, U1 RTL8221B-VB-CG, U2 STM32G031F6P6, U3 TPS62822DLC, U4 TPS22918DBVR, X1 MST8011AI-72-33E25

Commit message: References checked against the design; the fixes they turned up
docs/REFERENCES.md: the standards, Linux drivers, TI / Realtek / Microchip /
Gowin datasheets, app notes and EVMs, and commercial modules, each with a
table of the design against it.

Fixed from it:
- T1S: CLKHOLD_N (K3) tied high - pulled down during configuration, it would
  have held the flash clock and the FPGA would never load; P1 (also
  SSPI_CS_N) pulled up (R26); AN1718 BIN: 0.75 W end-node resistors (were
  0.25 W), 100 V centre cap (was 50 V), no copper under the CMC
- RJ45 / T1S: buck inductor 1.0 uH (TPS6282x Table 3): the RTL8221B wants
  its core switcher out of pulse skipping, which now starts at ~0.15 A, not
  ~0.33 A
- T1: no copper under the CMC on F/In1 (DP83TG720 8.5); the TC812 loadout
  fits the 200 uH CMC its datasheet asks for
- fw: PHY settings 70 ms after reset release (TG720: 65 ms before the first
  MDIO frame) with the 0x56 bridge answering 0xFFFF until then; LAN8670 set-up
  picked by silicon revision (AN1699 Rev G: C2 or D0); collision detection
  follows PLCA as AN1699 asks

All three boards: DRC 0 / 0 unconnected, KiCad 9 PASS, panels clean.
Parts:
- removed KiKit_MB_10_5, KiKit_MB_16_5, KiKit_MB_22_5, KiKit_MB_28_5, KiKit_MB_4_5: NPTH, NPTH
- added KiKit_MB_15_5: NPTH, NPTH, F.Cu at (157.8, 79.3)
- added KiKit_MB_21_5: NPTH, NPTH, F.Cu at (157.8, 98.3)
- added KiKit_MB_27_5: NPTH, NPTH, F.Cu at (157.8, 117.3)
- added KiKit_MB_3_5: NPTH, NPTH, F.Cu at (157.8, 41.3)
- added KiKit_MB_9_5: NPTH, NPTH, F.Cu at (157.8, 60.3)
- L1 (x5): value 470nH DFE201610E-R47M -> 1uH DFE201610E-1R0M
- moved KiKit_MB_15_1 25.3 mm to (160.9, 81.5)
- moved KiKit_MB_21_1 25.3 mm to (160.9, 100.5)
- moved KiKit_MB_27_1 25.3 mm to (160.9, 119.5)
- moved KiKit_MB_3_1 25.3 mm to (160.9, 43.5)
- moved KiKit_MB_9_1 25.3 mm to (160.9, 62.5)
- moved KiKit_MB_3_2 23.5 mm to (160.2, 42.8)
- moved KiKit_MB_15_2 23.5 mm to (160.2, 80.8)
- moved KiKit_MB_21_2 23.5 mm to (160.2, 99.8)
- moved KiKit_MB_27_2 23.5 mm to (160.2, 118.8)
- moved KiKit_MB_9_2 23.5 mm to (160.2, 61.8)
- moved KiKit_MB_3_3 21.7 mm to (159.5, 42.1)
- moved KiKit_MB_15_3 21.7 mm to (159.5, 80.1)
- moved KiKit_MB_21_3 21.7 mm to (159.5, 99.1)
- moved KiKit_MB_27_3 21.7 mm to (159.5, 118.1)
- moved KiKit_MB_9_3 21.7 mm to (159.5, 61.1)
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