File: hw/t1s/panel/t1s_panel.kicad_pcb (KiCad board)
At the start: 6 copper layers, 70 x 81 mm, 601 parts, among them J1 SFP edge (INF-8074i), J2 S2B-PH-K-S, U1 GW5AT-LV15MG132C1/I0, U2 GD25Q64CWIGR, U3 TPS62822DLC, U4 TPS22918DBVR, U5 LAN8670C2-E/LMX, U6 TLV75518PDBVR, U7 TLV75512PDBVR, U8 STM32G031F6P6, X1 OB2EL89CLIB112YLC-125M, Y1 25MHz CL12pF 2016

Commit message: References checked against the design; the fixes they turned up
docs/REFERENCES.md: the standards, Linux drivers, TI / Realtek / Microchip /
Gowin datasheets, app notes and EVMs, and commercial modules, each with a
table of the design against it.

Fixed from it:
- T1S: CLKHOLD_N (K3) tied high - pulled down during configuration, it would
  have held the flash clock and the FPGA would never load; P1 (also
  SSPI_CS_N) pulled up (R26); AN1718 BIN: 0.75 W end-node resistors (were
  0.25 W), 100 V centre cap (was 50 V), no copper under the CMC
- RJ45 / T1S: buck inductor 1.0 uH (TPS6282x Table 3): the RTL8221B wants
  its core switcher out of pulse skipping, which now starts at ~0.15 A, not
  ~0.33 A
- T1: no copper under the CMC on F/In1 (DP83TG720 8.5); the TC812 loadout
  fits the 200 uH CMC its datasheet asks for
- fw: PHY settings 70 ms after reset release (TG720: 65 ms before the first
  MDIO frame) with the 0x56 bridge answering 0xFFFF until then; LAN8670 set-up
  picked by silicon revision (AN1699 Rev G: C2 or D0); collision detection
  follows PLCA as AN1699 asks

All three boards: DRC 0 / 0 unconnected, KiCad 9 PASS, panels clean.
Parts:
- added R26: 4.7k, Resistor_SMD:R_0201_0603Metric, B.Cu at (154.2, 51.4)
- added R26: 4.7k, Resistor_SMD:R_0201_0603Metric, B.Cu at (154.2, 92.8)
- added R26: 4.7k, Resistor_SMD:R_0201_0603Metric, B.Cu at (154.2, 37.5)
- added R26: 4.7k, Resistor_SMD:R_0201_0603Metric, B.Cu at (154.2, 65.2)
- added R26: 4.7k, Resistor_SMD:R_0201_0603Metric, B.Cu at (154.2, 79.0)
- C42 (x5): value 100nF 50V -> 100nF 100V
- L1 (x5): value 470nH DFE201610E-R47M -> 1uH DFE201610E-1R0M
- R22 (x5), R23 (x5): value 49.9 1% -> 49.9 1% 0.75W
- moved KiKit_MB_14_4 35.9 mm to (159.0, 40.9)
- moved KiKit_MB_35_4 35.9 mm to (159.0, 82.3)
- moved KiKit_MB_7_4 35.9 mm to (159.0, 27.1)
- moved KiKit_MB_21_4 35.9 mm to (159.0, 54.7)
- moved KiKit_MB_28_4 35.9 mm to (159.0, 68.5)
- moved KiKit_MB_35_3 34.0 mm to (158.0, 82.3)
- moved KiKit_MB_14_3 34.0 mm to (158.0, 40.9)
- moved KiKit_MB_21_3 34.0 mm to (158.0, 54.7)
- moved KiKit_MB_28_3 34.0 mm to (158.0, 68.5)
- moved KiKit_MB_7_3 34.0 mm to (158.0, 27.1)
- moved KiKit_MB_14_2 32.2 mm to (157.0, 40.9)
- moved KiKit_MB_35_2 32.2 mm to (157.0, 82.3)
- moved KiKit_MB_7_2 32.2 mm to (157.0, 27.1)
- moved KiKit_MB_21_2 32.2 mm to (157.0, 54.7)
- moved KiKit_MB_28_2 32.2 mm to (157.0, 68.5)
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Connections:
- U1 pad K3: Board_0-unconnected-(U1-IOL26A-PadK3) -> Board_0-+3V3
- U1 pad K3: Board_4-unconnected-(U1-IOL26A-PadK3) -> Board_4-+3V3
- U1 pad K3: Board_3-unconnected-(U1-IOL26A-PadK3) -> Board_3-+3V3
- U1 pad K3: Board_1-unconnected-(U1-IOL26A-PadK3) -> Board_1-+3V3
- U1 pad K3: Board_2-unconnected-(U1-IOL26A-PadK3) -> Board_2-+3V3
Routing:
- net Board_4-+3V3: track 54.6 -> 55.6 mm, vias 33 -> 35
- net Board_0-+3V3: track 54.6 -> 55.6 mm, vias 33 -> 35
- net Board_3-+3V3: track 54.6 -> 55.6 mm, vias 33 -> 35
- net Board_2-+3V3: track 54.6 -> 55.6 mm, vias 33 -> 35
- net Board_1-+3V3: track 54.6 -> 55.6 mm, vias 33 -> 35
