File: hw/t1s/panel/t1s_panel.kicad_pcb (KiCad board)
At the start: 6 copper layers, 70 x 81 mm, 606 parts, among them J1 SFP edge (INF-8074i), J2 S2B-PH-K-S, U1 GW5AT-LV15MG132C1/I0, U2 GD25Q128EWIGR, U3 TPS62822DLC, U4 TPS22918DBVR, U5 LAN8670C2-E/LMX, U6 TLV75518PDBVR, U7 TLV75512PDBVR, U8 STM32G031F6P6, X1 OB2EL89CLIB112YLC-125M, Y1 25MHz CL12pF 2016

Commit message: T1S routed on the corrected SFP edge: DRC 0 / 0, KiCad 9 PASS, panel 0 errors
Freerouting for the slow nets around the hand-laid copper of 4687dd1, best
of two trials kept as t1s.ses (rebuild with --reuse-ses). Two links the
router left open, now laid before routing so any session gets them:
- a +3V3 via on C43's track for the MCU's VDD pin and its decaps (the old
  via sat where L2's current CMC land is);
- R8 / C14's core ends into In4's VCC_CORE island through their own via.

- KiCad 7: DRC 0 violations, 0 unconnected; ERC 0 errors (2 library-copy
  warnings, the LDOs, as before)
- KiCad 9: DRC 0 errors, 0 unconnected, parity clean, ERC 0 errors
- panel: 0 errors, 0 unconnected (library warnings only)
- edge: all 20 fingers as SFF-8419 figure 7-2, nets included
  (docs/COMPLIANCE.md section 3, positions stated independently)
- pairs: SRX 13.76/12.99 mm, no vias; STX 8.51/8.04 mm, 2/2 vias;
  both P to P

README: the edge-mirror warning is resolved for all three boards. T1S
stays "do not order" for its own reason - no transceiver IP, synthesis,
timing or bitstream yet.
Parts:
- removed the C1 at (122.5, 64.9)
- removed the C1 at (122.5, 51.1)
- removed the C1 at (122.5, 78.7)
- removed the C1 at (122.5, 37.3)
- removed the C1 at (122.5, 92.5)
- removed the C2 at (123.8, 51.1)
- removed the C2 at (123.8, 64.9)
- removed the C2 at (123.8, 78.7)
- removed the C2 at (123.8, 92.5)
- removed the C2 at (123.8, 37.3)
- removed the C3 at (118.7, 44.5)
- removed the C3 at (118.7, 30.7)
- removed the C3 at (118.7, 85.9)
- removed the C3 at (118.7, 58.3)
- removed the C3 at (118.7, 72.1)
- removed the C36 at (123.0, 28.1)
- removed the C36 at (123.0, 83.2)
- removed the C36 at (123.0, 69.5)
- removed the C36 at (123.0, 55.6)
- removed the C36 at (123.0, 41.9)
- removed the C37 at (119.7, 88.9)
- removed the C37 at (119.7, 33.7)
- removed the C37 at (119.7, 75.1)
- removed the C37 at (119.7, 61.3)
- removed the C37 at (119.7, 47.5)
- removed the C4 at (118.7, 29.9)
- removed the C4 at (118.7, 85.1)
- removed the C4 at (118.7, 57.5)
- removed the C4 at (118.7, 43.7)
- removed the C4 at (118.7, 71.3)
- removed the C5 at (118.7, 62.3)
- removed the C5 at (118.7, 48.5)
- removed the C5 at (118.7, 34.7)
- removed the C5 at (118.7, 76.1)
- removed the C5 at (118.7, 89.9)
- removed the C6 at (118.7, 76.9)
- removed the C6 at (118.7, 35.5)
- removed the C6 at (118.7, 63.1)
- removed the C6 at (118.7, 49.3)
- removed the C6 at (118.7, 90.7)
- removed the FB1 at (121.1, 45.7)
- removed the FB1 at (121.1, 59.5)
- removed the FB1 at (121.1, 73.3)
- removed the FB1 at (121.1, 31.9)
- removed the FB1 at (121.1, 87.1)
- removed the FB2 at (122.4, 51.6)
- removed the FB2 at (122.4, 79.2)
- removed the FB2 at (122.4, 37.8)
- removed the FB2 at (122.4, 93.0)
- removed the FB2 at (122.4, 65.4)
- removed the R1 at (124.2, 77.0)
- removed the R1 at (124.2, 90.8)
- removed the R1 at (124.2, 63.2)
- removed the R1 at (124.2, 35.6)
- removed the R1 at (124.2, 49.4)
- removed the R25 at (122.7, 31.0)
- removed the R25 at (122.7, 86.2)
- removed the R25 at (122.7, 44.8)
- removed the R25 at (122.7, 58.6)
- removed the R25 at (122.7, 72.4)
- removed the U4 at (120.5, 71.7)
- removed the U4 at (120.5, 57.9)
- removed the U4 at (120.5, 44.1)
- removed the U4 at (120.5, 85.5)
- removed the U4 at (120.5, 30.3)
- removed the U5 at (144.5, 60.5)
- removed the U5 at (144.5, 32.9)
- removed the U5 at (144.5, 74.3)
- removed the U5 at (144.5, 88.1)
- removed the U5 at (144.5, 46.7)
- added C1: 1uF, Capacitor_SMD:C_0402_1005Metric, B.Cu at (120.8, 73.2)
- added C1: 1uF, Capacitor_SMD:C_0402_1005Metric, B.Cu at (120.8, 59.4)
- added C1: 1uF, Capacitor_SMD:C_0402_1005Metric, B.Cu at (120.8, 87.0)
- added C1: 1uF, Capacitor_SMD:C_0402_1005Metric, B.Cu at (120.8, 31.8)
- added C1: 1uF, Capacitor_SMD:C_0402_1005Metric, B.Cu at (120.8, 45.6)
- added C2: 100nF, Capacitor_SMD:C_0402_1005Metric, B.Cu at (122.7, 87.0)
- added C2: 100nF, Capacitor_SMD:C_0402_1005Metric, B.Cu at (122.7, 59.4)
- added C2: 100nF, Capacitor_SMD:C_0402_1005Metric, B.Cu at (122.7, 73.2)
- added C2: 100nF, Capacitor_SMD:C_0402_1005Metric, B.Cu at (122.7, 31.8)
- added C2: 100nF, Capacitor_SMD:C_0402_1005Metric, B.Cu at (122.7, 45.6)
- added C3: 100nF, Capacitor_SMD:C_0201_0603Metric, F.Cu at (118.7, 62.7)
- added C3: 100nF, Capacitor_SMD:C_0201_0603Metric, F.Cu at (118.7, 90.3)
- added C3: 100nF, Capacitor_SMD:C_0201_0603Metric, F.Cu at (118.7, 76.5)
- added C3: 100nF, Capacitor_SMD:C_0201_0603Metric, F.Cu at (118.7, 48.9)
- added C3: 100nF, Capacitor_SMD:C_0201_0603Metric, F.Cu at (118.7, 35.1)
- added C36: 2.2nF, Capacitor_SMD:C_0402_1005Metric, F.Cu at (123.5, 50.6)
- added C36: 2.2nF, Capacitor_SMD:C_0402_1005Metric, F.Cu at (123.5, 64.4)
- added C36: 2.2nF, Capacitor_SMD:C_0402_1005Metric, F.Cu at (123.5, 92.0)
- added C36: 2.2nF, Capacitor_SMD:C_0402_1005Metric, F.Cu at (123.5, 36.8)
- added C36: 2.2nF, Capacitor_SMD:C_0402_1005Metric, F.Cu at (123.5, 78.2)
- added C37: 10uF, Capacitor_SMD:C_0402_1005Metric, F.Cu at (121.5, 78.4)
- added C37: 10uF, Capacitor_SMD:C_0402_1005Metric, F.Cu at (121.5, 50.8)
- added C37: 10uF, Capacitor_SMD:C_0402_1005Metric, F.Cu at (121.5, 37.0)
- added C37: 10uF, Capacitor_SMD:C_0402_1005Metric, F.Cu at (121.5, 64.6)
- added C37: 10uF, Capacitor_SMD:C_0402_1005Metric, F.Cu at (121.5, 92.2)
- added C4: 100nF, Capacitor_SMD:C_0201_0603Metric, F.Cu at (118.7, 91.1)
- added C4: 100nF, Capacitor_SMD:C_0201_0603Metric, F.Cu at (118.7, 35.9)
- added C4: 100nF, Capacitor_SMD:C_0201_0603Metric, F.Cu at (118.7, 63.5)
- added C4: 100nF, Capacitor_SMD:C_0201_0603Metric, F.Cu at (118.7, 77.3)
- added C4: 100nF, Capacitor_SMD:C_0201_0603Metric, F.Cu at (118.7, 49.7)
- added C5: 100nF, Capacitor_SMD:C_0201_0603Metric, F.Cu at (118.7, 58.7)
- added C5: 100nF, Capacitor_SMD:C_0201_0603Metric, F.Cu at (118.7, 86.3)
- added C5: 100nF, Capacitor_SMD:C_0201_0603Metric, F.Cu at (118.7, 72.5)
- added C5: 100nF, Capacitor_SMD:C_0201_0603Metric, F.Cu at (118.7, 44.9)
- added C5: 100nF, Capacitor_SMD:C_0201_0603Metric, F.Cu at (118.7, 31.1)
- added C6: 100nF, Capacitor_SMD:C_0201_0603Metric, F.Cu at (118.7, 44.1)
- added C6: 100nF, Capacitor_SMD:C_0201_0603Metric, F.Cu at (118.7, 71.7)
- added C6: 100nF, Capacitor_SMD:C_0201_0603Metric, F.Cu at (118.7, 85.5)
- added C6: 100nF, Capacitor_SMD:C_0201_0603Metric, F.Cu at (118.7, 30.3)
- added C6: 100nF, Capacitor_SMD:C_0201_0603Metric, F.Cu at (118.7, 57.9)
- added FB1: BLM18KG601SH1, Inductor_SMD:L_0603_1608Metric, F.Cu at (120.9, 88.8)
- added FB1: BLM18KG601SH1, Inductor_SMD:L_0603_1608Metric, F.Cu at (120.9, 33.6)
- added FB1: BLM18KG601SH1, Inductor_SMD:L_0603_1608Metric, F.Cu at (120.9, 75.0)
- added FB1: BLM18KG601SH1, Inductor_SMD:L_0603_1608Metric, F.Cu at (120.9, 47.5)
- added FB1: BLM18KG601SH1, Inductor_SMD:L_0603_1608Metric, F.Cu at (120.9, 61.2)
- added FB2: BLM18KG601SH1, Inductor_SMD:L_0603_1608Metric, F.Cu at (120.9, 73.4)
- added FB2: BLM18KG601SH1, Inductor_SMD:L_0603_1608Metric, F.Cu at (120.9, 59.6)
- added FB2: BLM18KG601SH1, Inductor_SMD:L_0603_1608Metric, F.Cu at (120.9, 45.8)
- added FB2: BLM18KG601SH1, Inductor_SMD:L_0603_1608Metric, F.Cu at (120.9, 32.0)
- added FB2: BLM18KG601SH1, Inductor_SMD:L_0603_1608Metric, F.Cu at (120.9, 87.2)
- added R1: 4.7k, Resistor_SMD:R_0201_0603Metric, B.Cu at (124.6, 36.5)
- added R1: 4.7k, Resistor_SMD:R_0201_0603Metric, B.Cu at (124.6, 50.2)
- added R1: 4.7k, Resistor_SMD:R_0201_0603Metric, B.Cu at (124.6, 77.8)
- added R1: 4.7k, Resistor_SMD:R_0201_0603Metric, B.Cu at (124.6, 91.7)
- added R1: 4.7k, Resistor_SMD:R_0201_0603Metric, B.Cu at (124.6, 64.0)
- added R25: 10k, Resistor_SMD:R_0201_0603Metric, B.Cu at (155.1, 79.0)
- added R25: 10k, Resistor_SMD:R_0201_0603Metric, B.Cu at (155.1, 51.4)
- added R25: 10k, Resistor_SMD:R_0201_0603Metric, B.Cu at (155.1, 92.8)
- added R25: 10k, Resistor_SMD:R_0201_0603Metric, B.Cu at (155.1, 37.5)
- added R25: 10k, Resistor_SMD:R_0201_0603Metric, B.Cu at (155.1, 65.2)
- added U4: TPS22918DBVR, Package_TO_SOT_SMD:SOT-23-6, B.Cu at (122.2, 35.9)
- added U4: TPS22918DBVR, Package_TO_SOT_SMD:SOT-23-6, B.Cu at (122.2, 77.3)
- added U4: TPS22918DBVR, Package_TO_SOT_SMD:SOT-23-6, B.Cu at (122.2, 91.1)
- added U4: TPS22918DBVR, Package_TO_SOT_SMD:SOT-23-6, B.Cu at (122.2, 63.5)
- added U4: TPS22918DBVR, Package_TO_SOT_SMD:SOT-23-6, B.Cu at (122.2, 49.7)
- added U5: LAN8670C2-E/LMX, Package_DFN_QFN:VQFN-32-1EP_5x5mm_P0.5mm_EP3.5x3.5mm, F.Cu at (144.5, 60.5)
- added U5: LAN8670C2-E/LMX, Package_DFN_QFN:VQFN-32-1EP_5x5mm_P0.5mm_EP3.5x3.5mm, F.Cu at (144.5, 32.9)
- added U5: LAN8670C2-E/LMX, Package_DFN_QFN:VQFN-32-1EP_5x5mm_P0.5mm_EP3.5x3.5mm, F.Cu at (144.5, 46.7)
- added U5: LAN8670C2-E/LMX, Package_DFN_QFN:VQFN-32-1EP_5x5mm_P0.5mm_EP3.5x3.5mm, F.Cu at (144.5, 88.1)
- added U5: LAN8670C2-E/LMX, Package_DFN_QFN:VQFN-32-1EP_5x5mm_P0.5mm_EP3.5x3.5mm, F.Cu at (144.5, 74.3)
- moved KiKit_MB_11_1 24.0 mm to (167.0, 40.9)
- moved KiKit_MB_11_2 24.0 mm to (168.0, 40.9)
- moved KiKit_MB_11_3 24.0 mm to (169.0, 40.9)
- moved KiKit_MB_11_4 24.0 mm to (170.0, 40.9)
- moved KiKit_MB_18_1 24.0 mm to (167.0, 54.7)
- moved KiKit_MB_18_2 24.0 mm to (168.0, 54.7)
- moved KiKit_MB_18_3 24.0 mm to (169.0, 54.7)
- moved KiKit_MB_18_4 24.0 mm to (170.0, 54.7)
- moved KiKit_MB_25_1 24.0 mm to (167.0, 68.5)
- moved KiKit_MB_25_2 24.0 mm to (168.0, 68.5)
- moved KiKit_MB_25_3 24.0 mm to (169.0, 68.5)
- moved KiKit_MB_25_4 24.0 mm to (170.0, 68.5)
- moved KiKit_MB_32_1 24.0 mm to (167.0, 82.3)
- moved KiKit_MB_32_2 24.0 mm to (168.0, 82.3)
- moved KiKit_MB_32_3 24.0 mm to (169.0, 82.3)
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Connections:
- U1 pad N1: Board_2-MODE1 -> Board_2-MODE
- U1 pad N2: Board_2-unconnected-(U1-IOL31B-PadN2) -> Board_2-MODE
- U1 pad N1: Board_0-MODE1 -> Board_0-MODE
- U1 pad N2: Board_0-unconnected-(U1-IOL31B-PadN2) -> Board_0-MODE
- U1 pad N1: Board_3-MODE1 -> Board_3-MODE
- U1 pad N2: Board_3-unconnected-(U1-IOL31B-PadN2) -> Board_3-MODE
- U1 pad N1: Board_1-MODE1 -> Board_1-MODE
- U1 pad N2: Board_1-unconnected-(U1-IOL31B-PadN2) -> Board_1-MODE
- U1 pad N1: Board_4-MODE1 -> Board_4-MODE
- U1 pad N2: Board_4-unconnected-(U1-IOL31B-PadN2) -> Board_4-MODE
- U8 pad 1: Board_4-SDA -> Board_4-SCL
- U8 pad 11: Board_4-unconnected-(U8-PA4-Pad11) -> Board_4-TX_FAULT
- U8 pad 12: Board_4-RX_LOS -> Board_4-unconnected-(U8-PA5-Pad12)
- U8 pad 13: Board_4-unconnected-(U8-PA6-Pad13) -> Board_4-TX_DISABLE
- U8 pad 17: Board_4-unconnected-(U8-PA12/PA10-Pad17) -> Board_4-SDA
- U8 pad 2: Board_4-TX_DISABLE -> Board_4-unconnected-(U8-PC14/PB9-Pad2)
- U8 pad 20: Board_4-SCL -> Board_4-unconnected-(U8-PB3/PB4/PB5/PB6-Pad20)
- U8 pad 3: Board_4-TX_FAULT -> Board_4-RX_LOS
- U8 pad 1: Board_1-SDA -> Board_1-SCL
- U8 pad 11: Board_1-unconnected-(U8-PA4-Pad11) -> Board_1-TX_FAULT
- U8 pad 12: Board_1-RX_LOS -> Board_1-unconnected-(U8-PA5-Pad12)
- U8 pad 13: Board_1-unconnected-(U8-PA6-Pad13) -> Board_1-TX_DISABLE
- U8 pad 17: Board_1-unconnected-(U8-PA12/PA10-Pad17) -> Board_1-SDA
- U8 pad 2: Board_1-TX_DISABLE -> Board_1-unconnected-(U8-PC14/PB9-Pad2)
- U8 pad 20: Board_1-SCL -> Board_1-unconnected-(U8-PB3/PB4/PB5/PB6-Pad20)
- U8 pad 3: Board_1-TX_FAULT -> Board_1-RX_LOS
- U8 pad 1: Board_2-SDA -> Board_2-SCL
- U8 pad 11: Board_2-unconnected-(U8-PA4-Pad11) -> Board_2-TX_FAULT
- U8 pad 12: Board_2-RX_LOS -> Board_2-unconnected-(U8-PA5-Pad12)
- U8 pad 13: Board_2-unconnected-(U8-PA6-Pad13) -> Board_2-TX_DISABLE
- U8 pad 17: Board_2-unconnected-(U8-PA12/PA10-Pad17) -> Board_2-SDA
- U8 pad 2: Board_2-TX_DISABLE -> Board_2-unconnected-(U8-PC14/PB9-Pad2)
- U8 pad 20: Board_2-SCL -> Board_2-unconnected-(U8-PB3/PB4/PB5/PB6-Pad20)
- U8 pad 3: Board_2-TX_FAULT -> Board_2-RX_LOS
- U8 pad 1: Board_3-SDA -> Board_3-SCL
- U8 pad 11: Board_3-unconnected-(U8-PA4-Pad11) -> Board_3-TX_FAULT
- U8 pad 12: Board_3-RX_LOS -> Board_3-unconnected-(U8-PA5-Pad12)
- U8 pad 13: Board_3-unconnected-(U8-PA6-Pad13) -> Board_3-TX_DISABLE
- U8 pad 17: Board_3-unconnected-(U8-PA12/PA10-Pad17) -> Board_3-SDA
- U8 pad 2: Board_3-TX_DISABLE -> Board_3-unconnected-(U8-PC14/PB9-Pad2)
- U8 pad 20: Board_3-SCL -> Board_3-unconnected-(U8-PB3/PB4/PB5/PB6-Pad20)
- U8 pad 3: Board_3-TX_FAULT -> Board_3-RX_LOS
- U8 pad 1: Board_0-SDA -> Board_0-SCL
- U8 pad 11: Board_0-unconnected-(U8-PA4-Pad11) -> Board_0-TX_FAULT
- U8 pad 12: Board_0-RX_LOS -> Board_0-unconnected-(U8-PA5-Pad12)
- U8 pad 13: Board_0-unconnected-(U8-PA6-Pad13) -> Board_0-TX_DISABLE
- U8 pad 17: Board_0-unconnected-(U8-PA12/PA10-Pad17) -> Board_0-SDA
- U8 pad 2: Board_0-TX_DISABLE -> Board_0-unconnected-(U8-PC14/PB9-Pad2)
- U8 pad 20: Board_0-SCL -> Board_0-unconnected-(U8-PB3/PB4/PB5/PB6-Pad20)
- U8 pad 3: Board_0-TX_FAULT -> Board_0-RX_LOS
Routing:
- net Board_1-MDC: track 12.3 -> 29.4 mm, vias 3 -> 2
- net Board_0-MDC: track 12.3 -> 29.4 mm, vias 3 -> 2
- net Board_3-MDC: track 12.3 -> 29.4 mm, vias 3 -> 2
- net Board_2-MDC: track 12.3 -> 29.4 mm, vias 3 -> 2
- net Board_4-MDC: track 12.3 -> 29.4 mm, vias 3 -> 2
- net Board_1-MDI_N: track 10.6 -> 22.9 mm
- net Board_4-MDI_N: track 10.6 -> 22.9 mm
- net Board_3-MDI_N: track 10.6 -> 22.9 mm
- net Board_0-MDI_N: track 10.6 -> 22.9 mm
- net Board_2-MDI_N: track 10.6 -> 22.9 mm
- net Board_2-TX_FAULT: track 39.2 -> 50.8 mm, vias 2 -> 3
- net Board_3-TX_FAULT: track 39.2 -> 50.8 mm, vias 2 -> 3
- net Board_1-TX_FAULT: track 39.2 -> 50.8 mm, vias 2 -> 3
- net Board_0-TX_FAULT: track 39.2 -> 50.8 mm, vias 2 -> 3
- net Board_4-TX_FAULT: track 39.2 -> 50.8 mm, vias 2 -> 3
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