File: hw/t1/t1.kicad_sch (KiCad schematic)
At the start: 66 parts, among them J1 SFP edge (INF-8074i), J2 Rosenberger E6S20A-40MT5-Z (H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, U1 DP83TG720S-Q1 (or DP83TC812S-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, U2 STM32G031F6P6, U3 TPS62822DLC, U4 TPS22918DBVR, Y1 25MHz CL8pF 2016

Commit message: T1: TI's OPEN Alliance MDI termination; bring-up order; honest README
- R6/R7 are now 1 k 1 % 0.75 W 2010 (RC2010FK-071KL), SNLA371B's
  configuration, along the board either side of the pair; the H-MTD and the
  board end moved 1 mm back (64.5 mm) to make the room. The unfitted 0402
  ESD footprints, not in TI's configuration, are gone.
- The DC block stays 100 nF 100 V X5R +-10 %: JLC stocks no SMD 1 % part
  at 100 V, nor a 0402 X7R (REFERENCES.md says so).
- Bottom-row escapes for VDDIO and LED0, a ground via for the decap pocket
  under U1, the TX pair 0.1 mm lower to let it in. DRC 0 / 0 unconnected,
  ERC 0, KiCad 9 PASS, panel 0 errors.
- ORDER.md: check pin 11/20 on the Gerbers; bring-up on a current-limited
  bench supply, then I2C 0x50/0x51/0x56, then one known host.
- README: what is SFP-standard and what is not (no SFF-8024 code for
  BASE-T1 / T1S; the EEPROM personality is a workaround), host SGMII and
  2500BASE-X requirements; RJ45/T1S marked do-not-order.
- COMPLIANCE.md regenerated: the independent edge check now fails RJ45/T1S.
Parts:
- removed D2, D3: ESD (DNP), Diode_SMD:D_0402_1005Metric, symbol Device:D_TVS
- R6, R7: value 1k 1% 0.2W -> 1k 1% 0.75W; footprint Resistor_SMD:R_0402_1005Metric -> Resistor_SMD:R_2010_5025Metric; LCSC C313354 -> C723477; MPN CRCW04021K00FKEDHP -> RC2010FK-071KL
