File: hw/t1s/t1s.kicad_sch (KiCad schematic)
At the start: 92 parts, among them J1 SFP edge (INF-8074i), J2 S2B-PH-K-S, U1 GW5AT-LV15MG132C1/I0, U2 GD25Q128EWIGR, U3 TPS62822DLC, U4 TPS22918DBVR, U5 LAN8670C2-E/LMX, U6 TLV75518PDBVR, U7 TLV75512PDBVR, U8 STM32G031F6P6, X1 OB2EL89CLIB112YLC-125M, Y1 25MHz CL12pF 2016

Commit message: T1S routed on the corrected SFP edge: DRC 0 / 0, KiCad 9 PASS, panel 0 errors
Freerouting for the slow nets around the hand-laid copper of 4687dd1, best
of two trials kept as t1s.ses (rebuild with --reuse-ses). Two links the
router left open, now laid before routing so any session gets them:
- a +3V3 via on C43's track for the MCU's VDD pin and its decaps (the old
  via sat where L2's current CMC land is);
- R8 / C14's core ends into In4's VCC_CORE island through their own via.

- KiCad 7: DRC 0 violations, 0 unconnected; ERC 0 errors (2 library-copy
  warnings, the LDOs, as before)
- KiCad 9: DRC 0 errors, 0 unconnected, parity clean, ERC 0 errors
- panel: 0 errors, 0 unconnected (library warnings only)
- edge: all 20 fingers as SFF-8419 figure 7-2, nets included
  (docs/COMPLIANCE.md section 3, positions stated independently)
- pairs: SRX 13.76/12.99 mm, no vias; STX 8.51/8.04 mm, 2/2 vias;
  both P to P

README: the edge-mirror warning is resolved for all three boards. T1S
stays "do not order" for its own reason - no transceiver IP, synthesis,
timing or bitstream yet.
Parts:
- C37: footprint Capacitor_SMD:C_0603_1608Metric -> Capacitor_SMD:C_0402_1005Metric; LCSC C19702 -> C15525
- U5: footprint Package_DFN_QFN:VQFN-32-1EP_5x5mm_P0.5mm_EP3.1x3.1mm -> Package_DFN_QFN:VQFN-32-1EP_5x5mm_P0.5mm_EP3.5x3.5mm
Connections:
- net MODE1 is gone; now on net MODE: R1.2, U1.N1 (IOL31A)
- net RX_LOS: now also U8.3 (PC15); no longer U8.12 (PA5)
- net SCL: now also U8.1 (PB7/PB8); no longer U8.20 (PB3/PB4/PB5/PB6)
- net SDA: now also U8.17 (PA12/PA10); no longer U8.1 (PB7/PB8)
- net SRX_M: now also C4.2; no longer C3.2
- net SRX_P: now also C3.2; no longer C4.2
- net TX_DISABLE: now also U8.13 (PA6); no longer U8.2 (PC14/PB9)
- net TX_FAULT: now also U8.11 (PA4); no longer U8.3 (PC15)
- net MODE: now reaches U1.N2 (IOL31B)
Changed lines of the file:
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@@
     (property "Reference" "C37" (at 178.03 247.19 0) (effects (font (size 1.0 1.0)) (justify left)))
     (property "Value" "10uF" (at 178.03 253.69 0) (effects (font (size 1.0 1.0)) (justify left)))
-    (property "Footprint" "Capacitor_SMD:C_0603_1608Metric" (at 176.53 250.19 0) (effects (font (size 1.0 1.0)) hide))
+    (property "Footprint" "Capacitor_SMD:C_0402_1005Metric" (at 176.53 250.19 0) (effects (font (size 1.0 1.0)) hide))
     (property "Datasheet" "" (at 176.53 250.19 0) (effects (font (size 1.0 1.0)) hide))
-    (property "LCSC" "C19702" (at 176.53 250.19 0) (effects (font (size 1.0 1.0)) hide))
+    (property "LCSC" "C15525" (at 176.53 250.19 0) (effects (font (size 1.0 1.0)) hide))
     (pin "1")
     (pin "2")
@@
     (property "Intersheetrefs" "${INTERSHEET_REFS}" (at 199.39 245.11 0) (effects (font (size 1.0 1.0)) hide)))
   (wire (pts (xy 199.39 252.73) (xy 199.39 255.27)) (stroke (width 0) (type default)))
-  (global_label "SRX_M" (shape passive) (at 199.39 255.27 270) (fields_autoplaced) (effects (font (size 1.0 1.0)) (justify right))
+  (global_label "SRX_P" (shape passive) (at 199.39 255.27 270) (fields_autoplaced) (effects (font (size 1.0 1.0)) (justify right))
     (property "Intersheetrefs" "${INTERSHEET_REFS}" (at 199.39 255.27 0) (effects (font (size 1.0 1.0)) hide)))
   (symbol (lib_id "Device:C_Small") (at 222.25 250.19 0) (unit 1)
@@
     (property "Intersheetrefs" "${INTERSHEET_REFS}" (at 222.25 245.11 0) (effects (font (size 1.0 1.0)) hide)))
   (wire (pts (xy 222.25 252.73) (xy 222.25 255.27)) (stroke (width 0) (type default)))
-  (global_label "SRX_P" (shape passive) (at 222.25 255.27 270) (fields_autoplaced) (effects (font (size 1.0 1.0)) (justify right))
+  (global_label "SRX_M" (shape passive) (at 222.25 255.27 270) (fields_autoplaced) (effects (font (size 1.0 1.0)) (justify right))
     (property "Intersheetrefs" "${INTERSHEET_REFS}" (at 222.25 255.27 0) (effects (font (size 1.0 1.0)) hide)))
   (symbol (lib_id "Device:C_Small") (at 245.11 250.19 0) (unit 1)
@@
     (property "Intersheetrefs" "${INTERSHEET_REFS}" (at 195.58 158.75 0) (effects (font (size 1.0 1.0)) hide)))
   (wire (pts (xy 193.04 163.83) (xy 195.58 163.83)) (stroke (width 0) (type default)))
-  (global_label "MODE1" (shape passive) (at 195.58 163.83 0) (fields_autoplaced) (effects (font (size 1.0 1.0)) (justify left))
+  (global_label "MODE" (shape passive) (at 195.58 163.83 0) (fields_autoplaced) (effects (font (size 1.0 1.0)) (justify left))
     (property "Intersheetrefs" "${INTERSHEET_REFS}" (at 195.58 163.83 0) (effects (font (size 1.0 1.0)) hide)))
+  (wire (pts (xy 193.04 179.07) (xy 195.58 179.07)) (stroke (width 0) (type default)))
+  (global_label "MODE" (shape passive) (at 195.58 179.07 0) (fields_autoplaced) (effects (font (size 1.0 1.0)) (justify left))
+    (property "Intersheetrefs" "${INTERSHEET_REFS}" (at 195.58 179.07 0) (effects (font (size 1.0 1.0)) hide)))
   (wire (pts (xy 193.04 199.39) (xy 195.58 199.39)) (stroke (width 0) (type default)))
   (global_label "FPGA_LINK" (shape passive) (at 195.58 199.39 0) (fields_autoplaced) (effects (font (size 1.0 1.0)) (justify left))
@@
   )
   (wire (pts (xy 359.41 252.73) (xy 359.41 255.27)) (stroke (width 0) (type default)))
-  (global_label "MODE1" (shape passive) (at 359.41 255.27 270) (fields_autoplaced) (effects (font (size 1.0 1.0)) (justify right))
+  (global_label "MODE" (shape passive) (at 359.41 255.27 270) (fields_autoplaced) (effects (font (size 1.0 1.0)) (justify right))
     (property "Intersheetrefs" "${INTERSHEET_REFS}" (at 359.41 255.27 0) (effects (font (size 1.0 1.0)) hide)))
   (symbol (lib_id "Device:R_Small") (at 39.37 273.05 0) (unit 1)
@@
     (property "Reference" "U5" (at 301.22 116.38 0) (effects (font (size 1.0 1.0)) (justify left)))
     (property "Value" "LAN8670C2-E/LMX" (at 301.22 122.88 0) (effects (font (size 1.0 1.0)) (justify left)))
-    (property "Footprint" "Package_DFN_QFN:VQFN-32-1EP_5x5mm_P0.5mm_EP3.1x3.1mm" (at 299.72 119.38 0) (effects (font (size 1.0 1.0)) hide))
+    (property "Footprint" "Package_DFN_QFN:VQFN-32-1EP_5x5mm_P0.5mm_EP3.5x3.5mm" (at 299.72 119.38 0) (effects (font (size 1.0 1.0)) hide))
     (property "Datasheet" "" (at 299.72 119.38 0) (effects (font (size 1.0 1.0)) hide))
     (property "MPN" "LAN8670C2-E/LMX" (at 299.72 119.38 0) (effects (font (size 1.0 1.0)) hide))
@@
   )
   (wire (pts (xy 279.40 232.41) (xy 276.86 232.41)) (stroke (width 0) (type default)))
-  (global_label "SDA" (shape passive) (at 276.86 232.41 180) (fields_autoplaced) (effects (font (size 1.0 1.0)) (justify right))
+  (global_label "SCL" (shape passive) (at 276.86 232.41 180) (fields_autoplaced) (effects (font (size 1.0 1.0)) (justify right))
     (property "Intersheetrefs" "${INTERSHEET_REFS}" (at 276.86 232.41 0) (effects (font (size 1.0 1.0)) hide)))
   (wire (pts (xy 320.04 222.25) (xy 322.58 222.25)) (stroke (width 0) (type default)))
   (global_label "PHY_INT_N" (shape passive) (at 322.58 222.25 0) (fields_autoplaced) (effects (font (size 1.0 1.0)) (justify left))
     (property "Intersheetrefs" "${INTERSHEET_REFS}" (at 322.58 222.25 0) (effects (font (size 1.0 1.0)) hide)))
-  (no_connect (at 320.04 224.79))
-  (wire (pts (xy 320.04 227.33) (xy 322.58 227.33)) (stroke (width 0) (type default)))
-  (global_label "RX_LOS" (shape passive) (at 322.58 227.33 0) (fields_autoplaced) (effects (font (size 1.0 1.0)) (justify left))
-    (property "Intersheetrefs" "${INTERSHEET_REFS}" (at 322.58 227.33 0) (effects (font (size 1.0 1.0)) hide)))
-  (no_connect (at 320.04 229.87))
+  (wire (pts (xy 320.04 224.79) (xy 322.58 224.79)) (stroke (width 0) (type default)))
+  (global_label "TX_FAULT" (shape passive) (at 322.58 224.79 0) (fields_autoplaced) (effects (font (size 1.0 1.0)) (justify left))
+    (property "Intersheetrefs" "${INTERSHEET_REFS}" (at 322.58 224.79 0) (effects (font (size 1.0 1.0)) hide)))
+  (no_connect (at 320.04 227.33))
+  (wire (pts (xy 320.04 229.87) (xy 322.58 229.87)) (stroke (width 0) (type default)))
+  (global_label "TX_DISABLE" (shape passive) (at 322.58 229.87 0) (fields_autoplaced) (effects (font (size 1.0 1.0)) (justify left))
+    (property "Intersheetrefs" "${INTERSHEET_REFS}" (at 322.58 229.87 0) (effects (font (size 1.0 1.0)) hide)))
   (wire (pts (xy 320.04 232.41) (xy 322.58 232.41)) (stroke (width 0) (type default)))
   (global_label "FPGA_LINK" (shape passive) (at 322.58 232.41 0) (fields_autoplaced) (effects (font (size 1.0 1.0)) (justify left))
@@
   (global_label "FPGA_DONE" (shape passive) (at 322.58 234.95 0) (fields_autoplaced) (effects (font (size 1.0 1.0)) (justify left))
     (property "Intersheetrefs" "${INTERSHEET_REFS}" (at 322.58 234.95 0) (effects (font (size 1.0 1.0)) hide)))
-  (no_connect (at 320.04 237.49))
+  (wire (pts (xy 320.04 237.49) (xy 322.58 237.49)) (stroke (width 0) (type default)))
+  (global_label "SDA" (shape passive) (at 322.58 237.49 0) (fields_autoplaced) (effects (font (size 1.0 1.0)) (justify left))
+    (property "Intersheetrefs" "${INTERSHEET_REFS}" (at 322.58 237.49 0) (effects (font (size 1.0 1.0)) hide)))
   (wire (pts (xy 320.04 240.03) (xy 322.58 240.03)) (stroke (width 0) (type default)))
   (global_label "SWDIO" (shape passive) (at 322.58 240.03 0) (fields_autoplaced) (effects (font (size 1.0 1.0)) (justify left))
@@
   (global_label "SWCLK" (shape passive) (at 322.58 242.57 0) (fields_autoplaced) (effects (font (size 1.0 1.0)) (justify left))
     (property "Intersheetrefs" "${INTERSHEET_REFS}" (at 322.58 242.57 0) (effects (font (size 1.0 1.0)) hide)))
-  (wire (pts (xy 279.40 219.71) (xy 276.86 219.71)) (stroke (width 0) (type default)))
-  (global_label "TX_DISABLE" (shape passive) (at 276.86 219.71 180) (fields_autoplaced) (effects (font (size 1.0 1.0)) (justify right))
-    (property "Intersheetrefs" "${INTERSHEET_REFS}" (at 276.86 219.71 0) (effects (font (size 1.0 1.0)) hide)))
-  (wire (pts (xy 279.40 229.87) (xy 276.86 229.87)) (stroke (width 0) (type default)))
-  (global_label "SCL" (shape passive) (at 276.86 229.87 180) (fields_autoplaced) (effects (font (size 1.0 1.0)) (justify right))
-    (property "Intersheetrefs" "${INTERSHEET_REFS}" (at 276.86 229.87 0) (effects (font (size 1.0 1.0)) hide)))
+  (no_connect (at 279.40 219.71))
+  (no_connect (at 279.40 229.87))
   (wire (pts (xy 279.40 222.25) (xy 276.86 222.25)) (stroke (width 0) (type default)))
-  (global_label "TX_FAULT" (shape passive) (at 276.86 222.25 180) (fields_autoplaced) (effects (font (size 1.0 1.0)) (justify right))
+  (global_label "RX_LOS" (shape passive) (at 276.86 222.25 180) (fields_autoplaced) (effects (font (size 1.0 1.0)) (justify right))
     (property "Intersheetrefs" "${INTERSHEET_REFS}" (at 276.86 222.25 0) (effects (font (size 1.0 1.0)) hide)))
   (wire (pts (xy 299.72 209.55) (xy 299.72 207.01)) (stroke (width 0) (type default)))
