File: hw/rj45/rj45.kicad_sch (KiCad schematic)
At the start: 67 parts, among them J1 SFP edge (INF-8074i), J2 KH-RJ45-58-8P8C, T1 LP72450ANL, U1 RTL8221B-VB-CG, U2 STM32G031F6P6, U3 TPS62822DLC, U4 TPS22918DBVR, X1 MST8011AI-72-33E25

Commit message: References checked against the design; the fixes they turned up
docs/REFERENCES.md: the standards, Linux drivers, TI / Realtek / Microchip /
Gowin datasheets, app notes and EVMs, and commercial modules, each with a
table of the design against it.

Fixed from it:
- T1S: CLKHOLD_N (K3) tied high - pulled down during configuration, it would
  have held the flash clock and the FPGA would never load; P1 (also
  SSPI_CS_N) pulled up (R26); AN1718 BIN: 0.75 W end-node resistors (were
  0.25 W), 100 V centre cap (was 50 V), no copper under the CMC
- RJ45 / T1S: buck inductor 1.0 uH (TPS6282x Table 3): the RTL8221B wants
  its core switcher out of pulse skipping, which now starts at ~0.15 A, not
  ~0.33 A
- T1: no copper under the CMC on F/In1 (DP83TG720 8.5); the TC812 loadout
  fits the 200 uH CMC its datasheet asks for
- fw: PHY settings 70 ms after reset release (TG720: 65 ms before the first
  MDIO frame) with the 0x56 bridge answering 0xFFFF until then; LAN8670 set-up
  picked by silicon revision (AN1699 Rev G: C2 or D0); collision detection
  follows PLCA as AN1699 asks

All three boards: DRC 0 / 0 unconnected, KiCad 9 PASS, panels clean.
Parts:
- L1: value 470nH DFE201610E-R47M -> 1uH DFE201610E-1R0M; LCSC C269773 -> C161082; MPN DFE201610E-R47M -> DFE201610E-1R0M
Changed lines of the file:
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@@
     (in_bom yes) (on_board yes) (dnp no)
     (property "Reference" "L1" (at 132.31 292.91 0) (effects (font (size 1.0 1.0)) (justify left)))
-    (property "Value" "470nH DFE201610E-R47M" (at 132.31 299.41 0) (effects (font (size 1.0 1.0)) (justify left)))
+    (property "Value" "1uH DFE201610E-1R0M" (at 132.31 299.41 0) (effects (font (size 1.0 1.0)) (justify left)))
     (property "Footprint" "Inductor_SMD:L_Murata_DFE201610P" (at 130.81 295.91 0) (effects (font (size 1.0 1.0)) hide))
     (property "Datasheet" "" (at 130.81 295.91 0) (effects (font (size 1.0 1.0)) hide))
-    (property "MPN" "DFE201610E-R47M" (at 130.81 295.91 0) (effects (font (size 1.0 1.0)) hide))
-    (property "LCSC" "C269773" (at 130.81 295.91 0) (effects (font (size 1.0 1.0)) hide))
+    (property "MPN" "DFE201610E-1R0M" (at 130.81 295.91 0) (effects (font (size 1.0 1.0)) hide))
+    (property "LCSC" "C161082" (at 130.81 295.91 0) (effects (font (size 1.0 1.0)) hide))
     (pin "1")
     (pin "2")

Commit message: RJ45 re-laid on the corrected SFP edge: U1 on top
With the edge drawn the right way round (SFF-8419 Figure 7-2) the RTL8221B's
SerDes pins meet RD-, RD+, TD+, TD- straight only from the top side; it has
no SerDes polarity swap. U1's group (decaps, straps, fan, oscillator, analog
beads, HSO caps) is turned over as one body in make_rj45.py; the links to
the rest are laid new:
- HSI and RD pairs on top, P to P, no via
- MDI on top under the magnetics' body straight into the chip-side pads,
  port 0 on channel 1; CFG_OPT1 now pulled down (no MDI swap)
- the slow lines laid on In2 end to end in the jack bus's lane order; the
  MCU's GPIOs follow it (fw VARIANT_RJ45: PA0 MDIO, PA1 MDC, PA4 TX_FAULT,
  PA5 TX_DISABLE, PA6 RX_LOS)
- both VCC beads, the load switch and its caps below the HSI pair; the
  buck's switch node under its own body; panel tabs moved off U4 and X1
DRC 0 / 0 unconnected, ERC 0, KiCad 9 PASS, panel 0 errors. T1S still
carries the mirrored edge.
Connections:
- net +3V3: no longer R13.1
- net GND: now also R13.1
- net MDC: now also U2.8 (PA1); no longer U2.7 (PA0)
- net MDI0_N: now also T1.3 (TD1-); no longer T1.11 (TD4+)
- net MDI0_P: now also T1.2 (TD1+); no longer T1.12 (TD4-)
- net MDI1_N: now also T1.6 (TD2-); no longer T1.8 (TD3+)
- net MDI1_P: now also T1.5 (TD2+); no longer T1.9 (TD3-)
- net MDI2_N: now also T1.9 (TD3-); no longer T1.5 (TD2+)
- net MDI2_P: now also T1.8 (TD3+); no longer T1.6 (TD2-)
- net MDI3_N: now also T1.12 (TD4-); no longer T1.2 (TD1+)
- net MDI3_P: now also T1.11 (TD4+); no longer T1.3 (TD1-)
- net MDIO: now also U2.7 (PA0); no longer U2.8 (PA1)
- net RX_LOS: now also U2.13 (PA6); no longer U2.12 (PA5)
- net TX_DISABLE: now also U2.12 (PA5); no longer U2.11 (PA4)
- net TX_FAULT: now also U2.11 (PA4); no longer U2.13 (PA6)
Changed lines of the file:
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@@
   )
   (wire (pts (xy 313.69 270.51) (xy 313.69 267.97)) (stroke (width 0) (type default)))
-  (symbol (lib_id "power:+3V3") (at 313.69 267.97 0) (unit 1)
-    (in_bom no) (on_board yes) (dnp no)
-    (property "Reference" "#PWR042" (at 315.19 264.97 0) (effects (font (size 1.0 1.0)) (justify left) hide))
-    (property "Value" "+3V3" (at 315.19 271.47 0) (effects (font (size 1.0 1.0)) (justify left) hide))
-    (property "Footprint" "" (at 313.69 267.97 0) (effects (font (size 1.0 1.0)) hide))
-    (property "Datasheet" "" (at 313.69 267.97 0) (effects (font (size 1.0 1.0)) hide))
+  (wire (pts (xy 313.69 267.97) (xy 313.69 270.51)) (stroke (width 0) (type default)))
+  (symbol (lib_id "power:GND") (at 313.69 270.51 0) (unit 1)
+    (in_bom no) (on_board yes) (dnp no)
+    (property "Reference" "#PWR042" (at 315.19 267.51 0) (effects (font (size 1.0 1.0)) (justify left) hide))
+    (property "Value" "GND" (at 315.19 274.01 0) (effects (font (size 1.0 1.0)) (justify left) hide))
+    (property "Footprint" "" (at 313.69 270.51 0) (effects (font (size 1.0 1.0)) hide))
+    (property "Datasheet" "" (at 313.69 270.51 0) (effects (font (size 1.0 1.0)) hide))
     (pin "1")
     (instances (project "rj45" (path "/3c9d2e71-5a4b-4f60-8d1e-7b2c3a4d5e61" (reference "#PWR042") (unit 1))))
@@
   )
   (wire (pts (xy 267.97 101.60) (xy 265.43 101.60)) (stroke (width 0) (type default)))
-  (global_label "MDI3_N" (shape passive) (at 265.43 101.60 180) (fields_autoplaced) (effects (font (size 1.0 1.0)) (justify right))
+  (global_label "MDI0_P" (shape passive) (at 265.43 101.60 180) (fields_autoplaced) (effects (font (size 1.0 1.0)) (justify right))
     (property "Intersheetrefs" "${INTERSHEET_REFS}" (at 265.43 101.60 0) (effects (font (size 1.0 1.0)) hide)))
   (wire (pts (xy 267.97 104.14) (xy 265.43 104.14)) (stroke (width 0) (type default)))
@@
     (property "Intersheetrefs" "${INTERSHEET_REFS}" (at 265.43 104.14 0) (effects (font (size 1.0 1.0)) hide)))
   (wire (pts (xy 267.97 106.68) (xy 265.43 106.68)) (stroke (width 0) (type default)))
-  (global_label "MDI3_P" (shape passive) (at 265.43 106.68 180) (fields_autoplaced) (effects (font (size 1.0 1.0)) (justify right))
+  (global_label "MDI0_N" (shape passive) (at 265.43 106.68 180) (fields_autoplaced) (effects (font (size 1.0 1.0)) (justify right))
     (property "Intersheetrefs" "${INTERSHEET_REFS}" (at 265.43 106.68 0) (effects (font (size 1.0 1.0)) hide)))
   (wire (pts (xy 267.97 109.22) (xy 265.43 109.22)) (stroke (width 0) (type default)))
-  (global_label "MDI2_N" (shape passive) (at 265.43 109.22 180) (fields_autoplaced) (effects (font (size 1.0 1.0)) (justify right))
+  (global_label "MDI1_P" (shape passive) (at 265.43 109.22 180) (fields_autoplaced) (effects (font (size 1.0 1.0)) (justify right))
     (property "Intersheetrefs" "${INTERSHEET_REFS}" (at 265.43 109.22 0) (effects (font (size 1.0 1.0)) hide)))
   (wire (pts (xy 267.97 111.76) (xy 265.43 111.76)) (stroke (width 0) (type default)))
@@
     (property "Intersheetrefs" "${INTERSHEET_REFS}" (at 265.43 111.76 0) (effects (font (size 1.0 1.0)) hide)))
   (wire (pts (xy 267.97 114.30) (xy 265.43 114.30)) (stroke (width 0) (type default)))
-  (global_label "MDI2_P" (shape passive) (at 265.43 114.30 180) (fields_autoplaced) (effects (font (size 1.0 1.0)) (justify right))
+  (global_label "MDI1_N" (shape passive) (at 265.43 114.30 180) (fields_autoplaced) (effects (font (size 1.0 1.0)) (justify right))
     (property "Intersheetrefs" "${INTERSHEET_REFS}" (at 265.43 114.30 0) (effects (font (size 1.0 1.0)) hide)))
   (wire (pts (xy 267.97 116.84) (xy 265.43 116.84)) (stroke (width 0) (type default)))
-  (global_label "MDI1_N" (shape passive) (at 265.43 116.84 180) (fields_autoplaced) (effects (font (size 1.0 1.0)) (justify right))
+  (global_label "MDI2_P" (shape passive) (at 265.43 116.84 180) (fields_autoplaced) (effects (font (size 1.0 1.0)) (justify right))
     (property "Intersheetrefs" "${INTERSHEET_REFS}" (at 265.43 116.84 0) (effects (font (size 1.0 1.0)) hide)))
   (wire (pts (xy 267.97 119.38) (xy 265.43 119.38)) (stroke (width 0) (type default)))
@@
     (property "Intersheetrefs" "${INTERSHEET_REFS}" (at 265.43 119.38 0) (effects (font (size 1.0 1.0)) hide)))
   (wire (pts (xy 267.97 121.92) (xy 265.43 121.92)) (stroke (width 0) (type default)))
-  (global_label "MDI1_P" (shape passive) (at 265.43 121.92 180) (fields_autoplaced) (effects (font (size 1.0 1.0)) (justify right))
+  (global_label "MDI2_N" (shape passive) (at 265.43 121.92 180) (fields_autoplaced) (effects (font (size 1.0 1.0)) (justify right))
     (property "Intersheetrefs" "${INTERSHEET_REFS}" (at 265.43 121.92 0) (effects (font (size 1.0 1.0)) hide)))
   (wire (pts (xy 267.97 124.46) (xy 265.43 124.46)) (stroke (width 0) (type default)))
-  (global_label "MDI0_N" (shape passive) (at 265.43 124.46 180) (fields_autoplaced) (effects (font (size 1.0 1.0)) (justify right))
+  (global_label "MDI3_P" (shape passive) (at 265.43 124.46 180) (fields_autoplaced) (effects (font (size 1.0 1.0)) (justify right))
     (property "Intersheetrefs" "${INTERSHEET_REFS}" (at 265.43 124.46 0) (effects (font (size 1.0 1.0)) hide)))
   (wire (pts (xy 267.97 127.00) (xy 265.43 127.00)) (stroke (width 0) (type default)))
@@
     (property "Intersheetrefs" "${INTERSHEET_REFS}" (at 265.43 127.00 0) (effects (font (size 1.0 1.0)) hide)))
   (wire (pts (xy 267.97 129.54) (xy 265.43 129.54)) (stroke (width 0) (type default)))
-  (global_label "MDI0_P" (shape passive) (at 265.43 129.54 180) (fields_autoplaced) (effects (font (size 1.0 1.0)) (justify right))
+  (global_label "MDI3_N" (shape passive) (at 265.43 129.54 180) (fields_autoplaced) (effects (font (size 1.0 1.0)) (justify right))
     (property "Intersheetrefs" "${INTERSHEET_REFS}" (at 265.43 129.54 0) (effects (font (size 1.0 1.0)) hide)))
   (wire (pts (xy 290.83 101.60) (xy 293.37 101.60)) (stroke (width 0) (type default)))
@@
     (property "Intersheetrefs" "${INTERSHEET_REFS}" (at 193.04 207.01 0) (effects (font (size 1.0 1.0)) hide)))
   (wire (pts (xy 190.50 209.55) (xy 193.04 209.55)) (stroke (width 0) (type default)))
-  (global_label "TX_DISABLE" (shape passive) (at 193.04 209.55 0) (fields_autoplaced) (effects (font (size 1.0 1.0)) (justify left))
+  (global_label "TX_FAULT" (shape passive) (at 193.04 209.55 0) (fields_autoplaced) (effects (font (size 1.0 1.0)) (justify left))
     (property "Intersheetrefs" "${INTERSHEET_REFS}" (at 193.04 209.55 0) (effects (font (size 1.0 1.0)) hide)))
   (wire (pts (xy 190.50 212.09) (xy 193.04 212.09)) (stroke (width 0) (type default)))
-  (global_label "RX_LOS" (shape passive) (at 193.04 212.09 0) (fields_autoplaced) (effects (font (size 1.0 1.0)) (justify left))
+  (global_label "TX_DISABLE" (shape passive) (at 193.04 212.09 0) (fields_autoplaced) (effects (font (size 1.0 1.0)) (justify left))
     (property "Intersheetrefs" "${INTERSHEET_REFS}" (at 193.04 212.09 0) (effects (font (size 1.0 1.0)) hide)))
   (wire (pts (xy 190.50 214.63) (xy 193.04 214.63)) (stroke (width 0) (type default)))
-  (global_label "TX_FAULT" (shape passive) (at 193.04 214.63 0) (fields_autoplaced) (effects (font (size 1.0 1.0)) (justify left))
+  (global_label "RX_LOS" (shape passive) (at 193.04 214.63 0) (fields_autoplaced) (effects (font (size 1.0 1.0)) (justify left))
     (property "Intersheetrefs" "${INTERSHEET_REFS}" (at 193.04 214.63 0) (effects (font (size 1.0 1.0)) hide)))
   (no_connect (at 190.50 217.17))
@@
     (property "Intersheetrefs" "${INTERSHEET_REFS}" (at 147.32 199.39 0) (effects (font (size 1.0 1.0)) hide)))
   (wire (pts (xy 190.50 199.39) (xy 193.04 199.39)) (stroke (width 0) (type default)))
-  (global_label "MDC" (shape passive) (at 193.04 199.39 0) (fields_autoplaced) (effects (font (size 1.0 1.0)) (justify left))
+  (global_label "MDIO" (shape passive) (at 193.04 199.39 0) (fields_autoplaced) (effects (font (size 1.0 1.0)) (justify left))
     (property "Intersheetrefs" "${INTERSHEET_REFS}" (at 193.04 199.39 0) (effects (font (size 1.0 1.0)) hide)))
   (wire (pts (xy 190.50 201.93) (xy 193.04 201.93)) (stroke (width 0) (type default)))
-  (global_label "MDIO" (shape passive) (at 193.04 201.93 0) (fields_autoplaced) (effects (font (size 1.0 1.0)) (justify left))
+  (global_label "MDC" (shape passive) (at 193.04 201.93 0) (fields_autoplaced) (effects (font (size 1.0 1.0)) (justify left))
     (property "Intersheetrefs" "${INTERSHEET_REFS}" (at 193.04 201.93 0) (effects (font (size 1.0 1.0)) hide)))
   (wire (pts (xy 190.50 204.47) (xy 193.04 204.47)) (stroke (width 0) (type default)))

Commit message: RJ45: PHY address straps on LED0/1/2, re-routed: DRC 0 / 0, KiCad 9 PASS, panel 0 errors
The RTL8221B's CONFIG pins have no internal pulls (datasheet 7.18), so
LED0/1/2 (PHYAD[2:0]) floated. R19-R21, 4.7k to ground: PHYAD 000, which the
PHY maps to address 1 (Table 16 note 2), the firmware's address. Three 0201s
above pins 33-35; C16 moved underneath its via, C17 0.3 mm west.

R11 (INT's pull-up) moved under INT's In2 via. Two links the router left
open are laid by hand before routing (VCCR finger to FB2 through In2, R4's
feedback end through In2); one fresh Freerouting session around them is
kept as rj45.ses.

sfpgen, for board rebuilds:
- plane_dogbones' no-room fallback no longer lays a pad-centre copy of a
  link the pad already has through hand-laid copper (it ran a +3V3 stub
  into the edge strip, and the n <= n0 DRC count let it through);
- drop_duplicate_plane_vias also drops GND router vias inside a locked GND
  via, and the later of two locked same-net vias on top of each other.

KiCad 7 DRC 0 / 0 unconnected, ERC 0; KiCad 9 DRC 0 errors, parity clean,
ERC 0 errors; panel 0 errors, 0 unconnected; edge pins as SFF-8419.
Parts:
- added R19, R20, R21: 4.7k, Resistor_SMD:R_0201_0603Metric, symbol Device:R_Small
Connections:
- net GND: now also R19.2, R20.2, R21.2
- net LED0: now reaches U1.33 (LED0/PHYAD0)
- net LED0: now also R19.1
- net LED1: now reaches U1.34 (LED1/PHYAD1)
- net LED1: now also R20.1
- net LED2: now reaches U1.35 (LED2/PHYAD2)
- net LED2: now also R21.1
- no-connect marks 17 -> 14
